File: eagle/esp_switch.sch (EAGLE design)
At the start: 22 parts, among them IC1 LT1117-3.3V, X1 MKDSN1,5/3-5,08

Commit message: update sch and brd
Parts:
- removed IC1: LT1117-3.3V, v-reg:LM317MB
- added U$1: LD1117, LD1117:LD1117
Connections:
- net 5V renamed N$3
- removed net N$3 (its old number): C1.2, C2.2, C3.2, D1.-, IC1.ADJ, JP1.1, LH1500.C, Q1.E, R1.1, RGBLED5MM.C, U$2.GND
- new net GND: C1.2, C2.2, C3.2, D1.-, JP1.1, LH1500.C, Q1.E, R1.1, RGBLED5MM.C, U$1.GND, U$2.GND
- net 3.3V: now also U$1.OUT; no longer IC1.OUT
- net N$6: now also U$1.IN; no longer IC1.IN
Changed lines of the file:
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@@
 <?xml version="1.0" encoding="utf-8"?>
 <!DOCTYPE eagle SYSTEM "eagle.dtd">
-<eagle version="8.0.2">
+<eagle version="8.0.1">
 <drawing>
 <settings>
@@
 <part name="JP1" library="jumper" deviceset="JP2E" device="" value="RS232_TTL"/>
 <part name="D1" library="rectifier" deviceset="B*S" device="" technology="6"/>
-<part name="IC1" library="v-reg" deviceset="LM317?*" device="MB" value="LT1117-3.3V"/>
 <part name="C1" library="eagle-ltspice" deviceset="C" device="" value="100n"/>
 <part name="C2" library="eagle-ltspice" deviceset="C" device="" value="4,7m"/>
@@
 <part name="LH1500" library="LH1500" deviceset="LH1500" device=""/>
 <part name="P+1" library="SparkFun" deviceset="3.3V" device=""/>
-<part name="U$4" library="SparkFun" deviceset="5V" device=""/>
 <part name="X1" library="con-phoenix-508" deviceset="MKDSN1,5/3-5,08" device=""/>
+<part name="GND1" library="supply1" deviceset="GND" device=""/>
+<part name="U$1" library="LD1117" deviceset="LD1117" device=""/>
 </parts>
 <sheets>
@@
 <instance part="JP1" gate="1" x="137.16" y="101.6" rot="R90"/>
 <instance part="D1" gate="G$1" x="73.66" y="83.82"/>
-<instance part="IC1" gate="G$1" x="104.14" y="83.82"/>
 <instance part="C1" gate="G$1" x="88.9" y="78.74"/>
 <instance part="C2" gate="G$1" x="124.46" y="78.74"/>
@@
 <instance part="LH1500" gate="G$1" x="60.96" y="127" rot="MR0"/>
 <instance part="P+1" gate="G$1" x="114.3" y="86.36"/>
-<instance part="U$4" gate="G$1" x="66.04" y="99.06"/>
 <instance part="X1" gate="-1" x="38.1" y="121.92" rot="R180"/>
 <instance part="X1" gate="-2" x="38.1" y="127" rot="R180"/>
 <instance part="X1" gate="-3" x="38.1" y="132.08" rot="R180"/>
+<instance part="GND1" gate="1" x="114.3" y="68.58"/>
+<instance part="U$1" gate="G$1" x="104.14" y="81.28"/>
 </instances>
 <busses>
@@
 <segment>
 <pinref part="D1" gate="G$1" pin="+"/>
-<pinref part="IC1" gate="G$1" pin="IN"/>
 <wire x1="78.74" y1="83.82" x2="81.28" y2="83.82" width="0.1524" layer="91"/>
 <pinref part="C1" gate="G$1" pin="1"/>
@@
 <wire x1="104.14" y1="139.7" x2="96.52" y2="139.7" width="0.1524" layer="91"/>
 <junction x="96.52" y="139.7"/>
+<pinref part="U$1" gate="G$1" pin="IN"/>
 </segment>
 </net>
@@
 </segment>
 </net>
-<net name="N$3" class="0">
+<net name="GND" class="0">
 <segment>
 <pinref part="LH1500" gate="G$1" pin="C"/>
@@
 <wire x1="83.82" y1="71.12" x2="88.9" y2="71.12" width="0.1524" layer="91"/>
 <wire x1="88.9" y1="71.12" x2="104.14" y2="71.12" width="0.1524" layer="91"/>
-<wire x1="104.14" y1="71.12" x2="124.46" y2="71.12" width="0.1524" layer="91"/>
+<wire x1="104.14" y1="71.12" x2="114.3" y2="71.12" width="0.1524" layer="91"/>
+<wire x1="114.3" y1="71.12" x2="124.46" y2="71.12" width="0.1524" layer="91"/>
 <wire x1="124.46" y1="71.12" x2="137.16" y2="71.12" width="0.1524" layer="91"/>
-<pinref part="IC1" gate="G$1" pin="ADJ"/>
 <wire x1="104.14" y1="76.2" x2="104.14" y2="71.12" width="0.1524" layer="91"/>
 <junction x="104.14" y="71.12"/>
@@
 <junction x="83.82" y="71.12"/>
 <junction x="83.82" y="109.22"/>
+<pinref part="GND1" gate="1" pin="GND"/>
+<junction x="114.3" y="71.12"/>
+<pinref part="U$1" gate="G$1" pin="GND"/>
 </segment>
 </net>
 <net name="3.3V" class="0">
 <segment>
-<pinref part="IC1" gate="G$1" pin="OUT"/>
 <wire x1="111.76" y1="83.82" x2="114.3" y2="83.82" width="0.1524" layer="91"/>
 <wire x1="114.3" y1="83.82" x2="124.46" y2="83.82" width="0.1524" layer="91"/>
@@
 <wire x1="114.3" y1="86.36" x2="114.3" y2="83.82" width="0.1524" layer="91"/>
 <junction x="114.3" y="83.82"/>
-</segment>
-</net>
-<net name="5V" class="0">
-<segment>
-<pinref part="AC_IN" gate="G$1" pin="3"/>
-<wire x1="58.42" y1="99.06" x2="66.04" y2="99.06" width="0.1524" layer="91"/>
-<pinref part="U$4" gate="G$1" pin="5V"/>
-<wire x1="66.04" y1="99.06" x2="66.04" y2="76.2" width="0.1524" layer="91"/>
-<junction x="66.04" y="99.06"/>
-<wire x1="66.04" y1="76.2" x2="73.66" y2="76.2" width="0.1524" layer="91"/>
-<pinref part="D1" gate="G$1" pin="AC2"/>
-<wire x1="73.66" y1="76.2" x2="73.66" y2="78.74" width="0.1524" layer="91"/>
+<pinref part="U$1" gate="G$1" pin="OUT"/>
 </segment>
 </net>
@@
 </segment>
 </net>
+<net name="N$3" class="0">
+<segment>
+<pinref part="AC_IN" gate="G$1" pin="3"/>
+<wire x1="58.42" y1="99.06" x2="66.04" y2="99.06" width="0.1524" layer="91"/>
+<wire x1="66.04" y1="99.06" x2="66.04" y2="76.2" width="0.1524" layer="91"/>
+<wire x1="66.04" y1="76.2" x2="73.66" y2="76.2" width="0.1524" layer="91"/>
+<pinref part="D1" gate="G$1" pin="AC2"/>
+<wire x1="73.66" y1="76.2" x2="73.66" y2="78.74" width="0.1524" layer="91"/>
+</segment>
+</net>

Commit message: changed AC power connector, optimized milling
Parts:
- AC_IN: value 5V AC -> (none); device con-jack:JACK-PLUG1 -> Wurth_Elektronik_Electromechanic_DC_Power_Jack_Connectors_rev16a_covek:694108301002
Connections:
- net N$1: now also AC_IN.2; no longer AC_IN.1
- net N$3: now also AC_IN.1; no longer AC_IN.3
Other:
- moved on the sheet: AC_IN
Changed lines of the file:
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@@
 <?xml version="1.0" encoding="utf-8"?>
 <!DOCTYPE eagle SYSTEM "eagle.dtd">
-<eagle version="8.0.1">
+<eagle version="8.0.2">
 <drawing>
 <settings>
@@
 <part name="U$2" library="diy-modules" deviceset="WIRELESS-WIFI-ESP-01" device=""/>
 <part name="FRAME1" library="frames" deviceset="A4L-LOC" device=""/>
-<part name="AC_IN" library="con-jack" deviceset="JACK-PLUG" device="1" value="5V AC"/>
 <part name="JP1" library="jumper" deviceset="JP2E" device="" value="RS232_TTL"/>
 <part name="D1" library="rectifier" deviceset="B*S" device="" technology="6"/>
@@
 <part name="GND1" library="supply1" deviceset="GND" device=""/>
 <part name="U$1" library="LD1117" deviceset="LD1117" device=""/>
+<part name="AC_IN" library="Wurth_Elektronik_Electromechanic_DC_Power_Jack_Connectors_rev16a_covek" deviceset="694108301002" device=""/>
 </parts>
 <sheets>
@@
 <instance part="U$2" gate="G$1" x="198.12" y="106.68"/>
 <instance part="FRAME1" gate="G$1" x="0" y="0"/>
-<instance part="AC_IN" gate="G$1" x="53.34" y="96.52"/>
 <instance part="JP1" gate="1" x="137.16" y="101.6" rot="R90"/>
 <instance part="D1" gate="G$1" x="73.66" y="83.82"/>
@@
 <instance part="GND1" gate="1" x="114.3" y="68.58"/>
 <instance part="U$1" gate="G$1" x="104.14" y="81.28"/>
+<instance part="AC_IN" gate="G$1" x="58.42" y="99.06"/>
 </instances>
 <busses>
@@
 <pinref part="D1" gate="G$1" pin="AC1"/>
 <wire x1="73.66" y1="88.9" x2="73.66" y2="93.98" width="0.1524" layer="91"/>
-<pinref part="AC_IN" gate="G$1" pin="1"/>
 <wire x1="73.66" y1="93.98" x2="58.42" y2="93.98" width="0.1524" layer="91"/>
+<pinref part="AC_IN" gate="G$1" pin="2"/>
 </segment>
 </net>
 <net name="N$3" class="0">
 <segment>
-<pinref part="AC_IN" gate="G$1" pin="3"/>
 <wire x1="58.42" y1="99.06" x2="66.04" y2="99.06" width="0.1524" layer="91"/>
 <wire x1="66.04" y1="99.06" x2="66.04" y2="76.2" width="0.1524" layer="91"/>
@@
 <pinref part="D1" gate="G$1" pin="AC2"/>
 <wire x1="73.66" y1="76.2" x2="73.66" y2="78.74" width="0.1524" layer="91"/>
-</segment>
-</net>
+<pinref part="AC_IN" gate="G$1" pin="1"/>
+</segment>
+</net>
